Commit message: allow set stiffness separately for each object

File: examples/sensors/tactile_pad_sensor.urdf (robot description, URDF)
Before this commit: robot tactile_sensor_pad, 3 links, 2 joints
Joints:
- joint elastomer_joint: axis (none) -> 0 0 1; limit (none) -> lower=-0.0001 upper=0.0001 effort=1000.0 velocity=0.01; type fixed -> prismatic
- joint elastomer_tip_joint: axis (none) -> 0 0 1; limit (none) -> lower=-0.0001 upper=0.0001 effort=1000.0 velocity=0.01; type fixed -> prismatic

Commit message: update

File: examples/sensors/tactile_pad_sensor.urdf (robot description, URDF)
Before this commit: robot tactile_sensor_pad, 3 links, 2 joints
Joints:
- joint elastomer_joint: axis 0 0 1 -> (none); limit lower=-0.0001 upper=0.0001 effort=1000.0 velocity=0.01 -> (none); type prismatic -> fixed
- joint elastomer_tip_joint: axis 0 0 1 -> (none); limit lower=-0.0001 upper=0.0001 effort=1000.0 velocity=0.01 -> (none); type prismatic -> fixed
