Commit message: update urdf

File: assets/wujihand-urdf/urdf/right.urdf (robot description, URDF)
Before this commit: robot wujihand-right-v1.0.0, 26 links, 25 joints
Links:
- link finger1_link2: geometry collision cylinder length=0.036 radius=0.009; visual mesh filename=package://wujihand-urdf/meshes/right/finger1_link2.STL
- link finger1_link3: geometry collision cylinder length=0.028 radius=0.009; visual mesh filename=package://wujihand-urdf/meshes/right/finger1_link3.STL
- link finger1_link4: geometry collision cylinder length=0.016 radius=0.009; visual mesh filename=package://wujihand-urdf/meshes/right/finger1_link4.STL
- link finger2_link2: geometry collision cylinder length=0.036 radius=0.009; visual mesh filename=package://wujihand-urdf/meshes/right/finger2_link2.STL
- link finger2_link3: geometry collision cylinder length=0.028 radius=0.009; visual mesh filename=package://wujihand-urdf/meshes/right/finger2_link3.STL
- link finger2_link4: geometry collision cylinder length=0.008 radius=0.009; visual mesh filename=package://wujihand-urdf/meshes/right/finger2_link4.STL
- link finger3_link2: geometry collision cylinder length=0.034 radius=0.009; visual mesh filename=package://wujihand-urdf/meshes/right/finger3_link2.STL
- link finger3_link3: geometry collision cylinder length=0.028 radius=0.009; visual mesh filename=package://wujihand-urdf/meshes/right/finger3_link3.STL
- link finger3_link4: geometry collision cylinder length=0.008 radius=0.009; visual mesh filename=package://wujihand-urdf/meshes/right/finger3_link4.STL
- link finger4_link2: geometry collision cylinder length=0.033 radius=0.009; visual mesh filename=package://wujihand-urdf/meshes/right/finger4_link2.STL
- link finger4_link3: geometry collision cylinder length=0.028 radius=0.009; visual mesh filename=package://wujihand-urdf/meshes/right/finger4_link3.STL
- link finger4_link4: geometry collision cylinder length=0.008 radius=0.009; visual mesh filename=package://wujihand-urdf/meshes/right/finger4_link4.STL
- link finger5_link2: geometry collision cylinder length=0.030 radius=0.009; visual mesh filename=package://wujihand-urdf/meshes/right/finger5_link2.STL
- link finger5_link3: geometry collision cylinder length=0.028 radius=0.009; visual mesh filename=package://wujihand-urdf/meshes/right/finger5_link3.STL
- link finger5_link4: geometry collision cylinder length=0.008 radius=0.009; visual mesh filename=package://wujihand-urdf/meshes/right/finger5_link4.STL
